File: VCF_MS-20/VCF_MS-20.kicad_pcb (KiCad board)
At the start: 2 copper layers, 55.9 x 96.5 mm, 42 parts, among them J1 POWER, J2 AUDIO IN, J3 AUDIO OUT, J4 CV IN, Q1 BC558, Q2 BC558, SW1/HPLP1 SW_DPDT_x2, SW2/OCT1 SW_SPDT/ATT, U1 LM324, U2 LM13700

Commit message: Update MS-20 VCO
Parts:
- R13: value 1.5k -> 2.2k
- R14: value 2.2k -> 1.5k
- R8: footprint Resistor_THT:R_Axial_DIN0207_L6.3mm_D2.5mm_P5.08mm_Vertical -> Potentiometer_THT:Potentiometer_Bourns_3386C_Horizontal
- moved R8 2.54 mm to (86.4, 43.2), turned to 0 degrees
- renumbered RV1/RESO1 to RV1, RV2/CV1 to RV2, RV3/FILT1 to RV3, RV4/LVL1 to RV4
Routing:
- net Net-(D1-K): track 27.9 -> 35.6 mm
- net Net-(D1-A): track 33.0 -> 38.1 mm

Commit message: Update pcb
Parts:
- C2: footprint Capacitor_THT:C_Rect_L9.0mm_W2.5mm_P7.50mm_MKT -> Capacitor_THT:C_Axial_L5.1mm_D3.1mm_P7.50mm_Horizontal
Changed lines of the file:
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@@
     )
   )
-  (footprint "Capacitor_THT:C_Rect_L9.0mm_W2.5mm_P7.50mm_MKT" (layer "F.Cu")
+  (footprint "Capacitor_THT:C_Axial_L5.1mm_D3.1mm_P7.50mm_Horizontal" (layer "F.Cu")
     (at 96.52 55.76 90)
-    (descr "C, Rect series, Radial, pin pitch=7.50mm, , length*width=9*2.5mm^2, Capacitor, https://en.tdk.eu/inf/20/20/db/fc_2009/MKT_B32560_564.pdf")
-    (tags "C Rect series Radial pin pitch 7.50mm  length 9mm width 2.5mm Capacitor")
+    (descr "C, Axial series, Axial, Horizontal, pin pitch=7.5mm, , length*diameter=5.1*3.1mm^2, http://www.vishay.com/docs/45231/arseries.pdf")
+    (tags "C Axial series Axial Horizontal pin pitch 7.5mm  length 5.1mm diameter 3.1mm")
     (property "Sheetfile" "VCF_MS-20.kicad_sch")
     (property "Sheetname" "")
@@
     (property "ki_keywords" "capacitor cap")
     (attr through_hole)
-    (fp_text reference "C2" (at 3.75 -2.5 90) (layer "F.SilkS")
+    (fp_text reference "C2" (at 3.75 -2.67 90) (layer "F.SilkS")
         (effects (font (size 1 1) (thickness 0.15)))
     )
-    (fp_text value "1.0n" (at 3.75 2.5 90) (layer "F.Fab")
+    (fp_text value "1.0n" (at 3.75 2.67 90) (layer "F.Fab")
         (effects (font (size 1 1) (thickness 0.15)))
     )
@@
         (effects (font (size 1 1) (thickness 0.15)))
     )
-    (fp_line (start -0.87 -1.37) (end -0.87 -0.665)
+    (fp_line (start 1.04 0) (end 1.08 0)
       (stroke (width 0.12) (type solid)) (layer "F.SilkS"))
-    (fp_line (start -0.87 -1.37) (end 8.37 -1.37)
+    (fp_line (start 1.08 -1.67) (end 1.08 1.67)
       (stroke (width 0.12) (type solid)) (layer "F.SilkS"))
-    (fp_line (start -0.87 0.665) (end -0.87 1.37)
+    (fp_line (start 1.08 1.67) (end 6.42 1.67)
       (stroke (width 0.12) (type solid)) (layer "F.SilkS"))
-    (fp_line (start -0.87 1.37) (end 8.37 1.37)
+    (fp_line (start 6.42 -1.67) (end 1.08 -1.67)
       (stroke (width 0.12) (type solid)) (layer "F.SilkS"))
-    (fp_line (start 8.37 -1.37) (end 8.37 -0.665)
+    (fp_line (start 6.42 1.67) (end 6.42 -1.67)
       (stroke (width 0.12) (type solid)) (layer "F.SilkS"))
-    (fp_line (start 8.37 0.665) (end 8.37 1.37)
+    (fp_line (start 6.46 0) (end 6.42 0)
       (stroke (width 0.12) (type solid)) (layer "F.SilkS"))
-    (fp_line (start -1.05 -1.5) (end -1.05 1.5)
+    (fp_line (start -1.05 -1.8) (end -1.05 1.8)
       (stroke (width 0.05) (type solid)) (layer "F.CrtYd"))
-    (fp_line (start -1.05 1.5) (end 8.55 1.5)
+    (fp_line (start -1.05 1.8) (end 8.55 1.8)
       (stroke (width 0.05) (type solid)) (layer "F.CrtYd"))
-    (fp_line (start 8.55 -1.5) (end -1.05 -1.5)
+    (fp_line (start 8.55 -1.8) (end -1.05 -1.8)
       (stroke (width 0.05) (type solid)) (layer "F.CrtYd"))
-    (fp_line (start 8.55 1.5) (end 8.55 -1.5)
+    (fp_line (start 8.55 1.8) (end 8.55 -1.8)
       (stroke (width 0.05) (type solid)) (layer "F.CrtYd"))
-    (fp_line (start -0.75 -1.25) (end -0.75 1.25)
+    (fp_line (start 0 0) (end 1.2 0)
       (stroke (width 0.1) (type solid)) (layer "F.Fab"))
-    (fp_line (start -0.75 1.25) (end 8.25 1.25)
+    (fp_line (start 1.2 -1.55) (end 1.2 1.55)
       (stroke (width 0.1) (type solid)) (layer "F.Fab"))
-    (fp_line (start 8.25 -1.25) (end -0.75 -1.25)
+    (fp_line (start 1.2 1.55) (end 6.3 1.55)
       (stroke (width 0.1) (type solid)) (layer "F.Fab"))
-    (fp_line (start 8.25 1.25) (end 8.25 -1.25)
+    (fp_line (start 6.3 -1.55) (end 1.2 -1.55)
+      (stroke (width 0.1) (type solid)) (layer "F.Fab"))
+    (fp_line (start 6.3 1.55) (end 6.3 -1.55)
+      (stroke (width 0.1) (type solid)) (layer "F.Fab"))
+    (fp_line (start 7.5 0) (end 6.3 0)
       (stroke (width 0.1) (type solid)) (layer "F.Fab"))
     (pad "1" thru_hole circle (at 0 0 90) (size 1.6 1.6) (drill 0.8) (layers "*.Cu" "*.Mask")
       (net 7 "Net-(U1B-+)") (pintype "passive"))
-    (pad "2" thru_hole circle (at 7.5 0 90) (size 1.6 1.6) (drill 0.8) (layers "*.Cu" "*.Mask")
+    (pad "2" thru_hole oval (at 7.5 0 90) (size 1.6 1.6) (drill 0.8) (layers "*.Cu" "*.Mask")
       (net 8 "Net-(D1-A)") (pintype "passive"))
-    (model "${KICAD6_3DMODEL_DIR}/Capacitor_THT.3dshapes/C_Rect_L9.0mm_W2.5mm_P7.50mm_MKT.wrl"
+    (model "${KICAD6_3DMODEL_DIR}/Capacitor_THT.3dshapes/C_Axial_L5.1mm_D3.1mm_P7.50mm_Horizontal.wrl"
       (offset (xyz 0 0 0))
       (scale (xyz 1 1 1))

Commit message: Update pcb
Parts:
- removed C9: 470n, Capacitor_THT:C_Disc_D5.0mm_W2.5mm_P5.00mm
- C1, C4, C5: footprint Capacitor_THT:C_Disc_D3.8mm_W2.6mm_P2.50mm -> Capacitor_THT:C_Disc_D4.7mm_W2.5mm_P5.00mm
- C3, C8: footprint Capacitor_THT:C_Disc_D5.0mm_W2.5mm_P5.00mm -> Capacitor_THT:C_Disc_D4.3mm_W1.9mm_P5.00mm
- C6: footprint Capacitor_THT:C_Rect_L9.0mm_W4.0mm_P7.50mm_MKT -> Capacitor_THT:C_Rect_L11.0mm_W3.5mm_P10.00mm_MKT
- R8: footprint Potentiometer_THT:Potentiometer_Bourns_3386C_Horizontal -> Potentiometer_THT:Potentiometer_Piher_PT-6-V_Vertical
- moved SW2/OCT1 35.9 mm to (116.8, 63.5), turned to 0 degrees
- moved C8 10.4 mm to (106.6, 68.6), turned to 180 degrees
- moved R8 5.61 mm to (81.3, 40.7), turned to -90 degrees
- moved C1 2.46 mm to (119.4, 45.8)
- moved C4 2.46 mm to (101.6, 35.6)
Connections:
- C8 pad 1: Net-(U1B--) -> Net-(SW2/OCT1-B)
- C8 pad 2: Net-(SW2/OCT1-C) -> Net-(J3-Pin_1)
- R5 pad 1: Net-(U1B--) -> Net-(SW2/OCT1-C)
- R6 pad 1: Net-(U1B--) -> Net-(SW2/OCT1-C)
- R7 pad 2: Net-(U1C--) -> Net-(SW2/OCT1-A)
- SW2/OCT1 pad 2: Net-(J3-Pin_1) -> Net-(SW2/OCT1-B)
- U1 pad 6: Net-(U1B--) -> Net-(SW2/OCT1-C)
- U1 pad 7: Net-(U1B--) -> Net-(SW2/OCT1-C)
- U1 pad 8: Net-(U1C--) -> Net-(SW2/OCT1-A)
- U1 pad 9: Net-(U1C--) -> Net-(SW2/OCT1-A)
Routing:
- net Net-(U1B--): track 43.2 -> 0.00 mm
- net Net-(SW2/OCT1-C): track 17.9 -> 48.3 mm
- net Net-(U1C--): track 28.0 -> 0.00 mm
- net Net-(SW2/OCT1-B): track 0.00 -> 12.7 mm
- net Net-(J3-Pin_1): track 93.5 -> 83.8 mm
- net Net-(SW2/OCT1-A): track 20.3 -> 25.4 mm
- net GND: track 269.1 -> 274.2 mm
- net Net-(J2-Pin_1): track 7.62 -> 10.1 mm
- net Net-(C1-Pad1): track 10.2 -> 12.6 mm
- net Net-(D1-A): track 38.1 -> 40.5 mm
- net Net-(R3-Pad1): track 66.0 -> 66.6 mm

Commit message: Update pcb
Parts:
- C1: footprint Capacitor_THT:C_Disc_D4.7mm_W2.5mm_P5.00mm -> Capacitor_THT:C_Rect_L9.0mm_W2.7mm_P7.50mm_MKT
- C2: footprint Capacitor_THT:C_Axial_L5.1mm_D3.1mm_P7.50mm_Horizontal -> Capacitor_THT:C_Rect_L9.0mm_W2.7mm_P7.50mm_MKT
- C3: footprint Capacitor_THT:C_Disc_D4.3mm_W1.9mm_P5.00mm -> Capacitor_THT:C_Rect_L9.0mm_W2.7mm_P7.50mm_MKT
- C6: footprint Capacitor_THT:C_Rect_L11.0mm_W3.5mm_P10.00mm_MKT -> Capacitor_THT:C_Rect_L11.0mm_W4.3mm_P10.00mm_MKT
- C8: footprint Capacitor_THT:C_Disc_D4.3mm_W1.9mm_P5.00mm -> Capacitor_THT:C_Rect_L9.0mm_W3.2mm_P7.50mm_MKT
- R12: footprint Resistor_THT:R_Axial_DIN0207_L6.3mm_D2.5mm_P7.62mm_Horizontal -> Resistor_THT:R_Axial_DIN0207_L6.3mm_D2.5mm_P10.16mm_Horizontal
- R8: footprint Potentiometer_THT:Potentiometer_Piher_PT-6-V_Vertical -> Potentiometer_THT:Potentiometer_Bourns_3296W_Vertical
- moved R8 55.9 mm to (137.2, 43.2), turned to 90 degrees
- moved C8 50.8 mm to (157.4, 68.6)
- moved R12 48.3 mm to (175.3, 53.3)
- moved C1 48.3 mm to (167.6, 48.3)
- moved C4 48.3 mm to (149.9, 35.6)
- moved U1 48.3 mm to (149.9, 48.3)
- moved U2 48.3 mm to (149.9, 78.7)
- moved C2 48.3 mm to (144.8, 55.8)
- moved J3 48.3 mm to (152.4, 116.8)
- moved Q1 48.3 mm to (172.7, 106.7)
- moved R1 48.3 mm to (144.8, 109.2)
- moved R11 48.3 mm to (162.6, 58.4)
- moved R13 48.3 mm to (134.6, 58.4)
- moved R15 48.3 mm to (144.8, 83.8)
- moved R16 48.3 mm to (134.6, 81.3)
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Routing:
- net GND: track 274.2 -> 266.6 mm
- net Net-(R3-Pad1): track 66.6 -> 61.6 mm
- net Net-(Q1-C): track 73.7 -> 78.6 mm
- net Net-(SW1/HPLP1A-C): track 15.3 -> 12.7 mm
- net Net-(SW2/OCT1-B): track 12.7 -> 10.2 mm
- net Net-(D1-A): track 40.5 -> 38.0 mm
- net Net-(C1-Pad1): track 12.6 -> 10.2 mm
